File: pcb/rxSD.brd (EAGLE design)
At the start: 20 x 40 mm, 8 parts, among them IC1 REG1117, IC2 STM32F042K6, J1 USB_A_PTH_MALE

Commit message: building it up
Parts:
- removed D1: RGB_LED_CA-150141M173100-R&G&B, nixx:3528-COMMON-ANODE
- removed IC1: REG1117, usbclogger:SOT223
- removed S1: SWITCH-MOMENTARY-2TURTLE, Adafruit Feather M0 Adalogger:KMR2
- added SD1: TF-HOLDER, clock:TF-PULL
- moved U$3 14.6 mm to (4.95, 43.8)
- moved E1 13.6 mm to (5.08, 48.3)
- moved IC2 6.63 mm to (10.0, 14.0)
Connections:
- net GND: no longer IC1.1
- net VDD: now also SD1.4
- net VSS: now also SD1.6
Other:
- board size 20 x 40 mm -> 20 x 55 mm
Changed lines of the file:
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@@
 <setting verticaltext="up"/>
 </settings>
-<grid distance="5" unitdist="mil" unit="mm" style="lines" multiple="1" display="no" altdistance="1" altunitdist="mil" altunit="mil"/>
+<grid distance="5" unitdist="mil" unit="mil" style="lines" multiple="1" display="no" altdistance="1" altunitdist="mil" altunit="mil"/>
 <layers>
 <layer number="1" name="Top" color="4" fill="1" visible="yes" active="yes"/>
@@
 <plain>
 <wire x1="0" y1="0" x2="20" y2="0" width="0" layer="20"/>
-<wire x1="20" y1="0" x2="20" y2="40" width="0" layer="20"/>
-<wire x1="20" y1="40" x2="0" y2="40" width="0" layer="20"/>
-<wire x1="0" y1="40" x2="0" y2="0" width="0" layer="20"/>
+<wire x1="20" y1="0" x2="20" y2="55" width="0" layer="20"/>
+<wire x1="20" y1="55" x2="0" y2="55" width="0" layer="20"/>
+<wire x1="0" y1="55" x2="0" y2="0" width="0" layer="20"/>
 </plain>
 <attributes>
@@
 </autorouter>
 <elements>
-<element name="U$3" library="nRF24L01-Chip-v13" package="QFN20_ALT1" value="NRF24L01ALT1" x="4.064" y="29.21"/>
+<element name="U$3" library="nRF24L01-Chip-v13" package="QFN20_ALT1" value="NRF24L01ALT1" x="4.953" y="43.815"/>
 <element name="J1" library="SparkFun-Connectors" package="USB-A-H" value="USB_A_PTH_MALE" x="10" y="3" rot="R90">
 <attribute name="PROD_ID" value="CONN-08367" x="10" y="3" size="1.778" layer="27" rot="R90" display="off"/>
 <attribute name="SF_ID" value="PRT-00437" x="10" y="3" size="1.778" layer="27" rot="R90" display="off"/>
 </element>
-<element name="IC2" library="nixx" package="TQFP32-08" value="STM32F042K6" x="11.397" y="20.447"/>
-<element name="E1" library="SparkFun-RF" package="TRACE_ANTENNA_2.4GHZ_15.2MM" value="ANTENNA-GROUNDEDTRACE-15.2MM" x="5.588" y="34.671"/>
+<element name="IC2" library="nixx" package="TQFP32-08" value="STM32F042K6" x="10" y="13.97"/>
+<element name="SD1" library="clock" package="TF-PULL" value="TF-HOLDER" x="9.492" y="31.242" rot="R90"/>
+<element name="E1" library="SparkFun-RF" package="TRACE_ANTENNA_2.4GHZ_15.2MM" value="ANTENNA-GROUNDEDTRACE-15.2MM" x="5.08" y="48.26"/>
 <element name="U$1" library="3pos_slide_switch" package="SW_3POS_FOOT_OFFICIAL" value="SW_3POS_DEVSW_3POS_OFFICIAL" x="0.508" y="19.558" rot="R270"/>
-<element name="IC1" library="usbclogger" package="SOT223" value="REG1117" x="11.176" y="10.795" rot="R90">
-<attribute name="MF" value="" x="-1.397" y="3.302" size="1.778" layer="27" rot="R90" display="off"/>
-<attribute name="MPN" value="REG1117" x="-1.397" y="3.302" size="1.778" layer="27" rot="R90" display="off"/>
-<attribute name="OC_FARNELL" value="1097566" x="-1.397" y="3.302" size="1.778" layer="27" rot="R90" display="off"/>
-<attribute name="OC_NEWARK" value="14P6981" x="-1.397" y="3.302" size="1.778" layer="27" rot="R90" display="off"/>
-</element>
-<element name="S1" library="Adafruit Feather M0 Adalogger" package="KMR2" value="SWITCH-MOMENTARY-2TURTLE" x="16.637" y="29.845" rot="R270"/>
-<element name="D1" library="nixx" package="3528-COMMON-ANODE" value="RGB_LED_CA-150141M173100-R&amp;G&amp;B" x="11.938" y="29.845" rot="R90"/>
 </elements>
 <signals>
@@
 <contactref element="U$3" pad="15"/>
 <contactref element="U$3" pad="18"/>
-<wire x1="4.064" y1="31.1354" x2="5.9894" y2="30.1963" width="0" layer="19" extent="1-1"/>
-<wire x1="3.5709" y1="27.2846" x2="5.9894" y2="30.1963" width="0" layer="19" extent="1-1"/>
+<contactref element="SD1" pad="4"/>
+<wire x1="4.953" y1="45.7404" x2="6.8784" y2="44.8013" width="0" layer="19" extent="1-1"/>
+<wire x1="4.4599" y1="41.8896" x2="6.8784" y2="44.8013" width="0" layer="19" extent="1-1"/>
+<wire x1="17.112" y1="32.342" x2="4.4599" y2="41.8896" width="0" layer="19" extent="1-1"/>
 </signal>
 <signal name="VDD_PA">
@@
 <contactref element="U$3" pad="17"/>
 <contactref element="U$3" pad="20"/>
-<wire x1="3.0777" y1="31.1354" x2="4.5571" y2="31.1354" width="0" layer="19" extent="1-1"/>
-<wire x1="4.064" y1="29.21" x2="4.5571" y2="31.1354" width="0" layer="19" extent="1-1"/>
-<wire x1="4.064" y1="27.2846" x2="4.064" y2="29.21" width="0" layer="19" extent="1-1"/>
-<wire x1="5.9894" y1="29.7031" x2="4.064" y2="29.21" width="0" layer="19" extent="1-1"/>
+<contactref element="SD1" pad="6"/>
+<wire x1="4.953" y1="41.8896" x2="4.953" y2="43.815" width="0" layer="19" extent="1-1"/>
+<wire x1="6.8784" y1="44.3081" x2="4.953" y2="43.815" width="0" layer="19" extent="1-1"/>
+<wire x1="5.4461" y1="45.7404" x2="4.953" y2="43.815" width="0" layer="19" extent="1-1"/>
+<wire x1="3.9667" y1="45.7404" x2="5.4461" y2="45.7404" width="0" layer="19" extent="1-1"/>
+<wire x1="17.112" y1="34.542" x2="4.953" y2="41.8896" width="0" layer="19" extent="1-1"/>
 </signal>
 <signal name="VBUS">
@@
 <signal name="GND">
 <contactref element="J1" pad="GND"/>
-<contactref element="IC1" pad="1"/>
-<wire x1="6.5" y1="5.4" x2="14.3256" y2="8.5344" width="0" layer="19" extent="1-1"/>
 </signal>
 </signals>
