File: pcb/rxSD.sch (EAGLE design)
At the start: 8 parts, among them IC1 REG1117, IC2 STM32F042K6, J1 USB_A_PTH_MALE

Commit message: building it up
Parts:
- removed D1: RGB_LED_CA-150141M173100-R&G&B, nixx:RGB_LED_CA-150141M173100-R&G&B
- removed IC1: REG1117, usbclogger:REG1117
- removed S1: SWITCH-MOMENTARY-2TURTLE, Adafruit Feather M0 Adalogger:SWITCH-MOMENTARY-2TURTLE
- added SD1: TF-HOLDER, clock:TF-HOLDER
Connections:
- removed net GND: IC1.GND
Changed lines of the file:
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@@
 <part name="J1" library="SparkFun-Connectors" deviceset="USB_A" device="_PTH_MALE"/>
 <part name="IC2" library="nixx" deviceset="STM32F042K6" device=""/>
+<part name="SD1" library="clock" deviceset="TF-HOLDER" device=""/>
 <part name="GND14" library="supply1" library_urn="urn:adsk.eagle:library:371" deviceset="GND" device=""/>
 <part name="+3V10" library="supply1" library_urn="urn:adsk.eagle:library:371" deviceset="+3V3" device=""/>
 <part name="E1" library="SparkFun-RF" deviceset="ANTENNA-GROUNDED" device="TRACE-15.2MM"/>
 <part name="U$1" library="3pos_slide_switch" deviceset="SW_3POS_DEV" device="SW_3POS_OFFICIAL"/>
-<part name="IC1" library="usbclogger" deviceset="REG1117" device=""/>
-<part name="GND2" library="clock" deviceset="GND" device=""/>
-<part name="S1" library="Adafruit Feather M0 Adalogger" deviceset="SWITCH-MOMENTARY-2" device="TURTLE"/>
-<part name="D1" library="nixx" deviceset="RGB_LED_CA" device="-150141M173100-R&amp;G&amp;B"/>
 </parts>
 <sheets>
@@
 <instance part="J1" gate="G$1" x="30.48" y="38.1"/>
 <instance part="IC2" gate="G$1" x="119.38" y="86.36"/>
+<instance part="SD1" gate="G$1" x="-63.5" y="27.94" rot="MR0"/>
 <instance part="GND14" gate="1" x="-68.58" y="7.62"/>
 <instance part="+3V10" gate="G$1" x="-81.28" y="33.02"/>
 <instance part="E1" gate="G$1" x="-20.32" y="43.18"/>
 <instance part="U$1" gate="G$1" x="-25.4" y="63.5"/>
-<instance part="IC1" gate="G$1" x="-30.48" y="2.54"/>
-<instance part="GND2" gate="1" x="-30.48" y="-12.7"/>
-<instance part="S1" gate="G$1" x="-53.34" y="25.4"/>
-<instance part="D1" gate="G$1" x="40.64" y="76.2"/>
 </instances>
 <busses>
 </busses>
 <nets>
-<net name="GND" class="0">
-<segment>
-<pinref part="IC1" gate="G$1" pin="GND"/>
-<pinref part="GND2" gate="1" pin="GND"/>
-</segment>
-</net>
 </nets>
 </sheet>
