File: pcb/tx.sch (EAGLE design)
At the start: 9 parts

Commit message: dt rx done
Parts:
- added BT1: (no value), SparkFun-Batteries:BATTERY-24.5MM_PTH
Changed lines of the file:
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@@
 <?xml version="1.0" encoding="utf-8"?>
 <!DOCTYPE eagle SYSTEM "eagle.dtd">
-<eagle version="9.1.0">
+<eagle version="9.1.3">
 <drawing>
 <settings>
-<setting alwaysvectorfont="no"/>
+<setting alwaysvectorfont="yes"/>
 <setting verticaltext="up"/>
 </settings>
@@
 <part name="U$7" library="L1" deviceset="M3_MOUNTING_HOLE" device=""/>
 <part name="U$8" library="L1" deviceset="M3_MOUNTING_HOLE" device=""/>
+<part name="BT1" library="SparkFun-Batteries" deviceset="BATTERY" device="-24.5MM_PTH"/>
 </parts>
 <sheets>
@@
 <instance part="U$7" gate="G$1" x="-30.48" y="-17.78"/>
 <instance part="U$8" gate="G$1" x="-45.72" y="-20.32"/>
+<instance part="BT1" gate="G$1" x="-53.34" y="43.18"/>
 </instances>
 <busses>

Commit message: before tx firmware test
Parts:
- added C1, C3: 100nF, clock:CAP0805
- added C10: 4.7µF, SparkFun-Passives:CAP0805
- added C11, C12: 4.7uF, clock:CAP0805
- added C2, C6: 2.2nF, clock:CAP0805
- added C4: 1.5pF, clock:CAP0805
- added C5: 1pF, clock:CAP0805
- added C7: 4.7pF, clock:CAP0805
- added C8, C9: 22pF, clock:CAP0805
- added D1, D2: BAT20J, SparkFun-DiscreteSemi:DIODE-SCHOTTKY-BAT20J
- added L1: 3.9nH, basicBoard:INDUCTOR0805
- added L2: 8.2nH, basicBoard:INDUCTOR0805
- added L3: 2.7nH, basicBoard:INDUCTOR0805
- added LED1: (no value), joyAnalog:LEDCHIP-LED0805
- added R1: 22K, joyAnalog:RESISTOR0805-RES
- added R2, R3: 5K1, joyAnalog:RESISTOR0805-RES
- added R4: 4.7K, SparkFun-Passives:RESISTOR0805-RES
- added R5: 27K, SparkFun-Passives:RESISTOR0805-RES
- added S2: (no value), Adafruit Feather M0 Adalogger:SWITCH-SPDT-SMD-A
- added U$9: XC6206_DEV, 3pos_slide_switch:XC6206_DEV
- added U3: MCP73831T-2ACI/OT, microbuilder:MCP73831/2
- added Y1: CRYSTAL-26MHZSMD-3.2X2.5, SparkFun-Clocks:CRYSTAL-26MHZSMD-3.2X2.5
- BT1: device SparkFun-Batteries:BATTERY-24.5MM_PTH -> tx:TX_SPARKFUN-BATTERIES_BATTERY-24.5MM_PTH
- U$1: value USBC_6P_DEV -> L1_USBC_6P_DEV; device L1:USBC_6P_DEV -> tx:L1_USBC_6P_DEV
Connections:
- new net +3V3: C1.1, C12.1, C2.1, U$3.VDD@15, U$3.VDD@18, U$3.VDD@7, U$9.OUT
- new net GND: BT1.+, C1.2, C10.2, C11.2, C12.2, C2.2, C3.2, C5.2, C6.2, C7.2, C8.2, C9.2, R1.2, R2.2, R3.2, R5.2, U$1.GND, U$3.VSS@0, U$3.VSS@14, U$3.VSS@17, U$3.VSS@20, U$3.VSS@8, U$9.GND, U3.VSS, Y1.3
- new net N$1: C3.1, U$3.DVDD
- new net N$10: R3.1, U$1.CC2
- new net N$11: R2.1, U$1.CC1
- new net N$12: LED1.C, R4.1
- new net N$13: R4.2, U3.STAT
- new net N$14: U$3.MOSI
- new net N$15: U$3.MISO
- new net N$16: U$3.SCK
- new net N$17: R5.1, U3.PROG
- new net N$19: D2.A, S2.P
- new net N$2: R1.1, U$3.IREF
- new net N$20: U$3.CSN
- new net N$21: U$3.CE
- new net N$25: BT1.-, C10.1, S2.S, U3.VBAT
- new net N$26: D1.A, U$1.VBUS
- new net N$27: C11.1, D1.C, D2.C, LED1.A, U$9.IN, U3.VDD
- new net N$3: L1.1, L2.1, U$3.ANT2
- new net N$4: C4.1, L1.2
- new net N$5: C4.2, C5.1
- new net N$6: L2.2, L3.1, U$3.ANT1
- new net N$7: C8.1, U$3.XC2, Y1.1
- new net N$8: C6.1, C7.1, L3.2, U$3.VDD_PA
- new net N$9: C9.1, U$3.XC1, Y1.2
Other:
- note added: "Charge current: I_CHG = 1000 / R_PROG"
- moved on the sheet: BT1, U$3

Commit message: tx before cleanup
Parts:
- added 4K7, R9: 22K, joyAnalog:RESISTOR0805-RES
- added C13: 100nF, clock:CAP0805
- added C14, C15: 4.7uF, clock:CAP0805
- added JP1: (no value), adafruit_changed:PINHD-1X3CB
- added LED2: (no value), joyAnalog:LEDCHIP-LED0805
- added R10, R11: 100K, SparkFun-Passives:RESISTOR0805-RES
- added R6, R7, R8: 27K, SparkFun-Passives:RESISTOR0805-RES
- added U$10: 324_SW, 3pos_slide_switch:324_SW
- added U$11: PINHD1X2, adafruit_changed:PINHD1X2
- S2: device Adafruit Feather M0 Adalogger:SWITCH-SPDT-SMD-A -> tx:SWITCH-SPDTTDFGDFG
Connections:
- new net N$18: R6.1, U$2.PA10, U1.SDA
- new net N$22: R7.1, U$2.PA9, U1.SCL
- new net N$23: R8.1, U$2.PF0/OSC_IN, U1.XSHUT
- new net N$24: U$2.PF1/OSC_OUT, U1.GPIO1
- new net N$28: 4K7.2, LED2.C
- new net N$29: LED2.A, U$2.PA1
- new net N$30: U$10.2, U$2.PA4
- new net N$31: JP1.3, U$2.PA13
- new net N$32: JP1.2, U$2.PA14
- new net N$33: JP1.1, U$2.PA2
- new net N$35: R10.1, R11.2, U$2.PA3
- net +3V3: now also C13.1, C14.1, C15.1, R6.2, R7.2, U$11.1, U$2.VDD, U$2.VDDA, U1.AVDD, U1.AVDDVCSEL
- net GND: now also 4K7.1, C13.2, C14.2, C15.2, R11.1, R8.2, R9.2, S2.GND, U$10.4, U$11.2, U$2.BOOT0, U$2.VSS, U$4.GND, U$4.GND@1, U1.AVSSVCSEL, U1.GND@1, U1.GND@2, U1.GND@3, U1.GND@4
- net N$14: now also U$2.PA7
- net N$15: now also U$2.PA6
- net N$16: now also U$2.PA5
- net N$20: now also U$2.PB1
- net N$21: now also R9.1, U$2.PA0
- net N$27: now also R10.2
- net N$5: now also U$4.FEED
Other:
- moved on the sheet: U$2, U1

Commit message: tx almost done
Parts:
- C14, C15: value 4.7uF -> 100nF
- R12: value 22K -> 4K7
- R6, R7, R8: value 27K -> 10K
- R9: value 22K -> 10K
- renumbered 4K7 to R12
Changed lines of the file:
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@@
 <part name="LED1" library="joyAnalog" deviceset="LED" device="CHIP-LED0805"/>
 <part name="GND18" library="clock" deviceset="GND" device=""/>
-<part name="R6" library="SparkFun-Passives" deviceset="RESISTOR" device="0805-RES" value="27K"/>
-<part name="R7" library="SparkFun-Passives" deviceset="RESISTOR" device="0805-RES" value="27K"/>
+<part name="R6" library="SparkFun-Passives" deviceset="RESISTOR" device="0805-RES" value="10K"/>
+<part name="R7" library="SparkFun-Passives" deviceset="RESISTOR" device="0805-RES" value="10K"/>
 <part name="+3V3" library="supply1" library_urn="urn:adsk.eagle:library:371" deviceset="+3V3" device=""/>
 <part name="+3V4" library="supply1" library_urn="urn:adsk.eagle:library:371" deviceset="+3V3" device=""/>
-<part name="R8" library="SparkFun-Passives" deviceset="RESISTOR" device="0805-RES" value="27K"/>
+<part name="R8" library="SparkFun-Passives" deviceset="RESISTOR" device="0805-RES" value="10K"/>
 <part name="+3V6" library="supply1" library_urn="urn:adsk.eagle:library:371" deviceset="+3V3" device=""/>
 <part name="GND19" library="clock" deviceset="GND" device=""/>
@@
 <part name="GND21" library="supply1" library_urn="urn:adsk.eagle:library:371" deviceset="GND" device=""/>
 <part name="GND22" library="supply1" library_urn="urn:adsk.eagle:library:371" deviceset="GND" device=""/>
-<part name="C14" library="clock" deviceset="CAP" device="0805" value="4.7uF"/>
-<part name="C15" library="clock" deviceset="CAP" device="0805" value="4.7uF"/>
+<part name="C14" library="clock" deviceset="CAP" device="0805" value="100nF"/>
+<part name="C15" library="clock" deviceset="CAP" device="0805" value="100nF"/>
 <part name="GND23" library="supply1" library_urn="urn:adsk.eagle:library:371" deviceset="GND" device=""/>
 <part name="GND24" library="supply1" library_urn="urn:adsk.eagle:library:371" deviceset="GND" device=""/>
 <part name="U$10" library="3pos_slide_switch" deviceset="324_SW" device=""/>
-<part name="R9" library="joyAnalog" deviceset="RESISTOR" device="0805-RES" value="22K"/>
+<part name="R9" library="joyAnalog" deviceset="RESISTOR" device="0805-RES" value="10K"/>
 <part name="GND25" library="supply1" library_urn="urn:adsk.eagle:library:371" deviceset="GND" device=""/>
 <part name="GND26" library="clock" deviceset="GND" device=""/>
 <part name="LED2" library="joyAnalog" deviceset="LED" device="CHIP-LED0805"/>
-<part name="4K7" library="joyAnalog" deviceset="RESISTOR" device="0805-RES" value="22K"/>
+<part name="R12" library="joyAnalog" deviceset="RESISTOR" device="0805-RES" value="4K7"/>
 <part name="GND27" library="supply1" library_urn="urn:adsk.eagle:library:371" deviceset="GND" device=""/>
 <part name="GND28" library="supply1" library_urn="urn:adsk.eagle:library:371" deviceset="GND" device=""/>
@@
 <instance part="GND26" gate="1" x="30.48" y="40.64"/>
 <instance part="LED2" gate="G$1" x="-10.16" y="-147.32" rot="R90"/>
-<instance part="4K7" gate="G$1" x="0" y="-147.32" rot="R180"/>
+<instance part="R12" gate="G$1" x="0" y="-147.32" rot="R180"/>
 <instance part="GND27" gate="1" x="7.62" y="-124.46"/>
 <instance part="GND28" gate="1" x="12.7" y="-149.86"/>
@@
 </segment>
 <segment>
-<pinref part="4K7" gate="G$1" pin="1"/>
+<pinref part="R12" gate="G$1" pin="1"/>
 <pinref part="GND28" gate="1" pin="GND"/>
 <wire x1="12.7" y1="-147.32" x2="5.08" y2="-147.32" width="0.1524" layer="91"/>
@@
 <segment>
 <pinref part="LED2" gate="G$1" pin="C"/>
-<pinref part="4K7" gate="G$1" pin="2"/>
-</segment>
-</net>
+<pinref part="R12" gate="G$1" pin="2"/>
+</segment>
+</net>

Commit message: cleanup
Parts:
- R12: value 4K7 -> 4.7K
- R2, R3: value 5K1 -> 5.1K
- R5: value 27K -> 22K
Changed lines of the file:
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@@
 <part name="Y1" library="SparkFun-Clocks" deviceset="CRYSTAL-26MHZ" device="SMD-3.2X2.5"/>
 <part name="GND6" library="supply1" deviceset="GND" device=""/>
-<part name="R3" library="joyAnalog" deviceset="RESISTOR" device="0805-RES" value="5K1"/>
-<part name="R2" library="joyAnalog" deviceset="RESISTOR" device="0805-RES" value="5K1"/>
+<part name="R3" library="joyAnalog" deviceset="RESISTOR" device="0805-RES" value="5.1K"/>
+<part name="R2" library="joyAnalog" deviceset="RESISTOR" device="0805-RES" value="5.1K"/>
 <part name="U3" library="microbuilder" deviceset="MCP73831/2" device="" value="MCP73831T-2ACI/OT"/>
 <part name="R4" library="SparkFun-Passives" deviceset="RESISTOR" device="0805-RES" value="4.7K"/>
 <part name="C10" library="SparkFun-Passives" deviceset="CAP" device="0805" value="4.7µF"/>
-<part name="R5" library="SparkFun-Passives" deviceset="RESISTOR" device="0805-RES" value="27K"/>
+<part name="R5" library="SparkFun-Passives" deviceset="RESISTOR" device="0805-RES" value="22K"/>
 <part name="GND7" library="supply1" library_urn="urn:adsk.eagle:library:371" deviceset="GND" device=""/>
 <part name="U$9" library="3pos_slide_switch" deviceset="XC6206_DEV" device=""/>
@@
 <part name="GND26" library="clock" deviceset="GND" device=""/>
 <part name="LED2" library="joyAnalog" deviceset="LED" device="CHIP-LED0805"/>
-<part name="R12" library="joyAnalog" deviceset="RESISTOR" device="0805-RES" value="4K7"/>
+<part name="R12" library="joyAnalog" deviceset="RESISTOR" device="0805-RES" value="4.7K"/>
 <part name="GND27" library="supply1" library_urn="urn:adsk.eagle:library:371" deviceset="GND" device=""/>
 <part name="GND28" library="supply1" library_urn="urn:adsk.eagle:library:371" deviceset="GND" device=""/>

Commit message: further cleanup
Parts:
- added SJ1, SJ2: JUMPER-SMT_2_NC_TRACE_NO-SILK, SparkFun-Jumpers:JUMPER-SMT_2_NC_TRACE_NO-SILK
Connections:
- new net N$34: SJ2.2, U$2.PF1/OSC_OUT
- net +3V3: now also R8.2, SJ1.1, SJ2.1
- net GND: now also U$10.1; no longer R8.2
- net N$21: now also U$2.PA4; no longer U$2.PA0
- net N$23: now also SJ1.2; no longer R8.1, U1.XSHUT
- net N$24: now also R8.1, U1.XSHUT; no longer U$2.PF1/OSC_OUT, U1.GPIO1
- net N$29: now also U$2.PA3; no longer U$2.PA1
- net N$30: now also U$10.3, U$2.PA0; no longer U$2.PA4
- net N$35: now also U$2.PA1; no longer U$2.PA3
Changed lines of the file:
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@@
 <part name="R9" library="joyAnalog" deviceset="RESISTOR" device="0805-RES" value="10K"/>
 <part name="GND25" library="supply1" library_urn="urn:adsk.eagle:library:371" deviceset="GND" device=""/>
-<part name="GND26" library="clock" deviceset="GND" device=""/>
 <part name="LED2" library="joyAnalog" deviceset="LED" device="CHIP-LED0805"/>
 <part name="R12" library="joyAnalog" deviceset="RESISTOR" device="0805-RES" value="4.7K"/>
@@
 <part name="GND30" library="supply1" library_urn="urn:adsk.eagle:library:371" deviceset="GND" device=""/>
 <part name="JP1" library="adafruit_changed" deviceset="PINHD-1X3" device="CB"/>
+<part name="+3V8" library="supply1" library_urn="urn:adsk.eagle:library:371" deviceset="+3V3" device=""/>
+<part name="SJ1" library="SparkFun-Jumpers" deviceset="JUMPER-SMT_2_NC_TRACE" device="_NO-SILK"/>
+<part name="SJ2" library="SparkFun-Jumpers" deviceset="JUMPER-SMT_2_NC_TRACE" device="_NO-SILK"/>
+<part name="+3V9" library="supply1" library_urn="urn:adsk.eagle:library:371" deviceset="+3V3" device=""/>
+<part name="+3V10" library="supply1" library_urn="urn:adsk.eagle:library:371" deviceset="+3V3" device=""/>
 </parts>
 <sheets>
@@
 <instance part="R9" gate="G$1" x="38.1" y="-48.26" rot="R270"/>
 <instance part="GND25" gate="1" x="38.1" y="-55.88"/>
-<instance part="GND26" gate="1" x="30.48" y="40.64"/>
 <instance part="LED2" gate="G$1" x="-10.16" y="-147.32" rot="R90"/>
 <instance part="R12" gate="G$1" x="0" y="-147.32" rot="R180"/>
@@
 <instance part="GND30" gate="1" x="-162.56" y="-71.12"/>
 <instance part="JP1" gate="A" x="22.86" y="-91.44" rot="R270"/>
+<instance part="+3V8" gate="G$1" x="25.4" y="45.72"/>
+<instance part="SJ1" gate="G$1" x="-48.26" y="-55.88"/>
+<instance part="SJ2" gate="G$1" x="-48.26" y="-66.04"/>
+<instance part="+3V9" gate="G$1" x="-58.42" y="-53.34"/>
+<instance part="+3V10" gate="G$1" x="-58.42" y="-63.5"/>
 </instances>
 <busses>
@@
 </segment>
 <segment>
-<pinref part="GND26" gate="1" pin="GND"/>
-<pinref part="R8" gate="G$1" pin="2"/>
-<wire x1="30.48" y1="43.18" x2="25.4" y2="43.18" width="0.1524" layer="91"/>
-</segment>
-<segment>
 <pinref part="U$10" gate="G$1" pin="4"/>
 <pinref part="GND27" gate="1" pin="GND"/>
+<pinref part="U$10" gate="G$1" pin="1"/>
+<wire x1="7.62" y1="-121.92" x2="-22.86" y2="-121.92" width="0.1524" layer="91"/>
+<junction x="7.62" y="-121.92"/>
 </segment>
 <segment>
@@
 <wire x1="40.64" y1="-129.54" x2="50.8" y2="-129.54" width="0.1524" layer="91"/>
 </segment>
+<segment>
+<pinref part="R8" gate="G$1" pin="2"/>
+<pinref part="+3V8" gate="G$1" pin="+3V3"/>
+</segment>
+<segment>
+<pinref part="+3V9" gate="G$1" pin="+3V3"/>
+<pinref part="SJ1" gate="G$1" pin="1"/>
+<wire x1="-58.42" y1="-55.88" x2="-53.34" y2="-55.88" width="0.1524" layer="91"/>
+</segment>
+<segment>
+<pinref part="+3V10" gate="G$1" pin="+3V3"/>
+<pinref part="SJ2" gate="G$1" pin="1"/>
+<wire x1="-58.42" y1="-66.04" x2="-53.34" y2="-66.04" width="0.1524" layer="91"/>
+</segment>
 </net>
 <net name="N$1" class="0">
@@
 <pinref part="U$3" gate="G$1" pin="CE"/>
 <wire x1="76.2" y1="-53.34" x2="60.96" y2="-53.34" width="0.1524" layer="91"/>
-<pinref part="U$2" gate="G$1" pin="PA0"/>
 <wire x1="60.96" y1="-53.34" x2="60.96" y2="-43.18" width="0.1524" layer="91"/>
-<wire x1="60.96" y1="-43.18" x2="38.1" y2="-43.18" width="0.1524" layer="91"/>
+<wire x1="60.96" y1="-43.18" x2="43.18" y2="-43.18" width="0.1524" layer="91"/>
 <pinref part="R9" gate="G$1" pin="1"/>
-<wire x1="38.1" y1="-43.18" x2="5.08" y2="-43.18" width="0.1524" layer="91"/>
+<wire x1="43.18" y1="-43.18" x2="38.1" y2="-43.18" width="0.1524" layer="91"/>
+<pinref part="U$2" gate="G$1" pin="PA4"/>
+<wire x1="5.08" y1="-53.34" x2="30.48" y2="-53.34" width="0.1524" layer="91"/>
+<wire x1="30.48" y1="-53.34" x2="30.48" y2="-43.18" width="0.1524" layer="91"/>
+<wire x1="30.48" y1="-43.18" x2="38.1" y2="-43.18" width="0.1524" layer="91"/>
 <junction x="38.1" y="-43.18"/>
 </segment>
@@
 </segment>
 </net>
-<net name="N$23" class="0">
-<segment>
-<pinref part="U1" gate="G$1" pin="XSHUT"/>
-<pinref part="R8" gate="G$1" pin="1"/>
-<wire x1="30.48" y1="33.02" x2="25.4" y2="33.02" width="0.1524" layer="91"/>
-<wire x1="25.4" y1="33.02" x2="25.4" y2="-27.94" width="0.1524" layer="91"/>
-<wire x1="25.4" y1="-27.94" x2="-50.8" y2="-27.94" width="0.1524" layer="91"/>
-<junction x="25.4" y="33.02"/>
-<pinref part="U$2" gate="G$1" pin="PF0/OSC_IN"/>
-<wire x1="-50.8" y1="-27.94" x2="-50.8" y2="-55.88" width="0.1524" layer="91"/>
-<wire x1="-50.8" y1="-55.88" x2="-33.02" y2="-55.88" width="0.1524" layer="91"/>
-</segment>
-</net>
-<net name="N$24" class="0">
-<segment>
-<pinref part="U1" gate="G$1" pin="GPIO1"/>
-<wire x1="30.48" y1="30.48" x2="27.94" y2="30.48" width="0.1524" layer="91"/>
-<wire x1="27.94" y1="30.48" x2="27.94" y2="-25.4" width="0.1524" layer="91"/>
-<wire x1="27.94" y1="-25.4" x2="-55.88" y2="-25.4" width="0.1524" layer="91"/>
-<pinref part="U$2" gate="G$1" pin="PF1/OSC_OUT"/>
-<wire x1="-55.88" y1="-25.4" x2="-55.88" y2="-66.04" width="0.1524" layer="91"/>
-<wire x1="-55.88" y1="-66.04" x2="-33.02" y2="-66.04" width="0.1524" layer="91"/>
-</segment>
-</net>
 <net name="N$28" class="0">
 <segment>
 <pinref part="LED2" gate="G$1" pin="C"/>
 <pinref part="R12" gate="G$1" pin="2"/>
-</segment>
-</net>
-<net name="N$29" class="0">
-<segment>
-<pinref part="U$2" gate="G$1" pin="PA1"/>
-<wire x1="5.08" y1="-45.72" x2="-12.7" y2="-45.72" width="0.1524" layer="91"/>
-<wire x1="-12.7" y1="-45.72" x2="-12.7" y2="-144.78" width="0.1524" layer="91"/>
-<pinref part="LED2" gate="G$1" pin="A"/>
-<wire x1="-12.7" y1="-144.78" x2="-12.7" y2="-147.32" width="0.1524" layer="91"/>
-</segment>
-</net>
-<net name="N$30" class="0">
-<segment>
-<pinref part="U$2" gate="G$1" pin="PA4"/>
-<wire x1="5.08" y1="-53.34" x2="-12.7" y2="-53.34" width="0.1524" layer="91"/>
-<pinref part="U$10" gate="G$1" pin="2"/>
-<wire x1="-12.7" y1="-53.34" x2="-22.86" y2="-53.34" width="0.1524" layer="91"/>
-<wire x1="-22.86" y1="-53.34" x2="-22.86" y2="-114.3" width="0.1524" layer="91"/>
 </segment>
 </net>
@@
 <pinref part="R11" gate="G$1" pin="2"/>
 <wire x1="-162.56" y1="-55.88" x2="-162.56" y2="-53.34" width="0.1524" layer="91"/>
-<pinref part="U$2" gate="G$1" pin="PA3"/>
 <wire x1="-162.56" y1="-53.34" x2="-162.56" y2="-48.26" width="0.1524" layer="91"/>
-<wire x1="5.08" y1="-50.8" x2="-20.32" y2="-50.8" width="0.1524" layer="91"/>
-<wire x1="-20.32" y1="-50.8" x2="-20.32" y2="-48.26" width="0.1524" layer="91"/>
+<wire x1="-152.4" y1="-53.34" x2="-162.56" y2="-53.34" width="0.1524" layer="91"/>
+<junction x="-162.56" y="-53.34"/>
+<pinref part="U$2" gate="G$1" pin="PA1"/>
+<wire x1="5.08" y1="-45.72" x2="-20.32" y2="-45.72" width="0.1524" layer="91"/>
+<wire x1="-20.32" y1="-45.72" x2="-20.32" y2="-48.26" width="0.1524" layer="91"/>
 <wire x1="-20.32" y1="-48.26" x2="-152.4" y2="-48.26" width="0.1524" layer="91"/>
 <wire x1="-152.4" y1="-48.26" x2="-152.4" y2="-53.34" width="0.1524" layer="91"/>
-<wire x1="-152.4" y1="-53.34" x2="-162.56" y2="-53.34" width="0.1524" layer="91"/>
-<junction x="-162.56" y="-53.34"/>
 </segment>
 </net>
@@
 </segment>
 </net>
+<net name="N$24" class="0">
+<segment>
+<pinref part="R8" gate="G$1" pin="1"/>
+<pinref part="U1" gate="G$1" pin="XSHUT"/>
+<wire x1="30.48" y1="33.02" x2="25.4" y2="33.02" width="0.1524" layer="91"/>
+</segment>
+</net>
+<net name="N$23" class="0">
+<segment>
+<pinref part="U$2" gate="G$1" pin="PF0/OSC_IN"/>
+<pinref part="SJ1" gate="G$1" pin="2"/>
+<wire x1="-33.02" y1="-55.88" x2="-43.18" y2="-55.88" width="0.1524" layer="91"/>
+</segment>
+</net>
+<net name="N$34" class="0">
+<segment>
+<pinref part="SJ2" gate="G$1" pin="2"/>
+<wire x1="-43.18" y1="-66.04" x2="-35.56" y2="-66.04" width="0.1524" layer="91"/>
+<pinref part="U$2" gate="G$1" pin="PF1/OSC_OUT"/>
+<wire x1="-35.56" y1="-66.04" x2="-33.02" y2="-66.04" width="0.1524" layer="91"/>
+</segment>
+</net>
+<net name="N$29" class="0">
+<segment>
+<pinref part="U$2" gate="G$1" pin="PA3"/>
+<pinref part="LED2" gate="G$1" pin="A"/>
+<wire x1="5.08" y1="-50.8" x2="-12.7" y2="-50.8" width="0.1524" layer="91"/>
+<wire x1="-12.7" y1="-50.8" x2="-12.7" y2="-147.32" width="0.1524" layer="91"/>
+</segment>
+</net>
+<net name="N$30" class="0">
+<segment>
+<pinref part="U$2" gate="G$1" pin="PA0"/>
+<pinref part="U$10" gate="G$1" pin="2"/>
+<wire x1="5.08" y1="-43.18" x2="-22.86" y2="-43.18" width="0.1524" layer="91"/>
+<wire x1="-22.86" y1="-43.18" x2="-22.86" y2="-114.3" width="0.1524" layer="91"/>
+<pinref part="U$10" gate="G$1" pin="3"/>
+<wire x1="-22.86" y1="-114.3" x2="7.62" y2="-114.3" width="0.1524" layer="91"/>
+<junction x="-22.86" y="-114.3"/>
+</segment>
+</net>
