File: pcb/rx.sch (EAGLE design)
At the start: 34 parts, among them IC1 STM32F042F4, IC2 NRF24L01ALT1, SW1 SW_3POS_DEVSW_3POS_OFFICIAL, SW2 324_SW324_SWITCH_FOOT_HOLE, U1 USBC_16P_CENTERED, U2 XC6206_DEV, Y1 16MHz_12pF

Commit message: updated USBC connector, check_battery DBZ
Parts:
- U1: value USBC_16P_CENTERED -> USBC_16P; device my_usbc_16p_centered:USBC_16P_CENTERED -> my_usbc_16p:USBC_16P
Changed lines of the file:
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@@
 <part name="C14" library="clock" deviceset="CAP" device="0805" value="4.7uF"/>
 <part name="TP2" library="testpad" library_urn="urn:adsk.eagle:library:385" deviceset="TP" device="TP12R" package3d_urn="urn:adsk.eagle:package:27963/1"/>
-<part name="U1" library="my_usbc_16p_centered" deviceset="USBC_16P_CENTERED" device=""/>
+<part name="U1" library="my_usbc_16p" deviceset="USBC_16P" device=""/>
 <part name="SW1" library="3pos_slide_switch_centered" deviceset="SW_3POS_DEV" device="SW_3POS_OFFICIAL"/>
 </parts>
