File: pcb/AAA/rx_usba.brd (EAGLE design)
At the start: 19 x 38 mm, 32 parts, among them Y1 CRYSTAL-26MHZSMD-3.2X2.5

Commit message: txrx rev2 finished
Parts:
- removed R3, R5: 5.1K, joyAnalog:0805
- removed U$6: USBC_16P, my_usbc_16p:USBC_16P_FOOT
- added J1: USB_A_PTH_MALE, rx20:USB-A-H
- moved U$1 3.07 mm to (0.58, 15.8)
- moved C1 2.79 mm to (1.91, 20.5)
- moved C10 2.79 mm to (14.9, 7.59)
- moved C11 2.79 mm to (8.66, 7.84)
- moved C2 2.79 mm to (1.91, 22.2)
- moved C3 2.79 mm to (1.91, 18.9)
- moved C7 2.79 mm to (9.53, 24.6)
- moved C8 2.79 mm to (13.9, 18.9)
- moved C9 2.79 mm to (10.5, 22.9)
- moved E1 2.79 mm to (4.95, 29.8)
- moved L1 2.79 mm to (5.21, 25.5)
- moved L2 2.79 mm to (6.10, 23.2)
- moved L3 2.79 mm to (6.99, 25.5)
- moved R1 2.79 mm to (1.91, 23.8)
- moved R2 2.79 mm to (17.1, 18.9)
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Connections:
- removed net N$25: R3.1, U$6.B5
- removed net N$27: R5.1, U$6.A5
- net +5V: now also J1.VBUS; no longer U$6.A4B9, U$6.B4A9
- net GND: now also J1.GND, J1.SHLD1, J1.SHLD2; no longer R3.2, R5.2, U$6.A1B12, U$6.B11A12, U$6.P$13, U$6.P$14, U$6.P$15, U$6.P$16
- net N$12: now also J1.D-; no longer U$6.A7, U$6.B7
- net N$13: now also J1.D+; no longer U$6.A6, U$6.B6
Routing:
- net +5V: track 28.7 -> 5.76 mm
- net N$27: track 11.5 -> 0.00 mm
- net GND: track 41.9 -> 31.4 mm
- net N$25: track 6.90 -> 0.00 mm
- net N$26: track 12.4 -> 17.6 mm
- net N$10: track 15.1 -> 10.1 mm
- net N$13: track 11.4 -> 7.13 mm, vias 2 -> 0
- net N$12: track 11.2 -> 8.54 mm
- net +3V3: track 28.5 -> 29.4 mm
Other:
- board size 19 x 38 mm -> 19 x 35 mm
- board text removed: "REV2 FEB19"
