File: pcb/v2_experimental/no_transistor/tx.brd (EAGLE design)
At the start: 28 x 36.5 mm, 53 parts, among them IC1 STM32F030F4, IC2 NRF24L01ALT1, SW2 324_SW324_SWITCH_FOOT_HOLE, U2 USBC_16P, U3 MCP73831T-2ACI/OT, U4 XC6206_DEV, Y1 16MHz_12pF

Commit message: added a testpad
Parts:
- added TP2: TPTP10R, testpad:TP10R
Connections:
- net N$36: now also TP2.TP
Routing:
- net N$36: track 19.4 -> 20.2 mm
Changed lines of the file:
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@@
 <element name="U$14" library="3pos_slide_switch" package="M2_SCREW_FOOT" value="M2_SCREW_DEV" x="25.5" y="27" smashed="yes"/>
 <element name="R14" library="joyAnalog" package="0805" value="1 Ohm" x="23.9014" y="20.4216" smashed="yes" rot="R180">
-<attribute name="NAME" x="25.2857" y="17.7292" size="0.8128" layer="25" rot="R90"/>
-<attribute name="VALUE" x="24.9174" y="21.8186" size="0.4064" layer="27" rot="R180"/>
-<attribute name="VALUE" x="24.9174" y="21.8186" size="0.4064" layer="27" rot="R180"/>
+<attribute name="NAME" x="24.511" y="22.9997" size="0.8128" layer="25" rot="R180"/>
 </element>
 <element name="U2" library="my_usbc_16p" package="USBC_16P_FOOT" value="USBC_16P" x="14" y="3.8481" smashed="yes"/>
+<element name="TP2" library="testpad" library_urn="urn:adsk.eagle:library:385" package="TP10R" package3d_urn="urn:adsk.eagle:package:27959/1" value="TPTP10R" x="12.3952" y="15.0114" smashed="yes" rot="MR0">
+<attribute name="POPULARITY" value="3" x="12.3952" y="15.0114" size="1.778" layer="28" rot="MR0" display="off"/>
+<attribute name="TP_SIGNAL_NAME" value="" x="12.3952" y="15.0114" size="1.778" layer="28" rot="MR0" display="off"/>
+<attribute name="VALUE" x="12.7762" y="14.5034" size="0.0254" layer="28" rot="MR0"/>
+</element>
 </elements>
 <signals>
@@
 <wire x1="11.43" y1="14.8082" x2="11.43" y2="15.9766" width="0.1524" layer="16"/>
 <wire x1="21.4884" y1="12.9032" x2="13.335" y2="12.9032" width="0.1524" layer="16"/>
-<wire x1="13.335" y1="12.9032" x2="11.43" y2="14.8082" width="0.1524" layer="16"/>
+<wire x1="13.335" y1="12.9032" x2="11.811" y2="14.4272" width="0.1524" layer="16"/>
+<wire x1="11.811" y1="14.4272" x2="11.43" y2="14.8082" width="0.1524" layer="16"/>
 <wire x1="14.8" y1="14.6" x2="14.8" y2="15.045" width="0.1524" layer="1"/>
 <wire x1="14.478" y1="15.367" x2="14.8" y2="15.045" width="0.1524" layer="1"/>
@@
 <wire x1="13.2588" y1="15.5956" x2="13.4874" y2="15.367" width="0.1524" layer="1"/>
 <wire x1="13.4874" y1="15.367" x2="14.478" y2="15.367" width="0.1524" layer="1"/>
+<contactref element="TP2" pad="TP"/>
+<wire x1="12.3952" y1="15.0114" x2="11.811" y2="14.4272" width="0.1524" layer="16"/>
 </signal>
 </signals>
@@
 which will not be processed correctly with this version.
 </note>
+<note version="8.2" severity="warning">
+Since Version 8.2, EAGLE supports online libraries. The ids
+of those online libraries will not be understood (or retained)
+with this version.
+</note>
+<note version="8.3" severity="warning">
+Since Version 8.3, EAGLE supports URNs for individual library
+assets (packages, symbols, and devices). The URNs of those assets
+will not be understood (or retained) with this version.
+</note>
+<note version="8.3" severity="warning">
+Since Version 8.3, EAGLE supports the association of 3D packages
+with devices in libraries, schematics, and board files. Those 3D
+packages will not be understood (or retained) with this version.
+</note>
 </compatibility>
