File: pcb/v2_experimental/no_transistor/tx.sch (EAGLE design)
At the start: 53 parts, among them IC1 STM32F030F4, IC2 NRF24L01ALT1, SW2 324_SW324_SWITCH_FOOT_HOLE, U2 USBC_16P, U3 MCP73831T-2ACI/OT, U4 XC6206_DEV, Y1 16MHz_12pF

Commit message: added a testpad
Parts:
- added TP2: TPTP10R, testpad:TPTP10R
Connections:
- net N$36: now also TP2.TP
Changed lines of the file:
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@@
 <part name="R14" library="joyAnalog" deviceset="RESISTOR" device="0805-RES" value="1 Ohm"/>
 <part name="U2" library="my_usbc_16p" deviceset="USBC_16P" device=""/>
+<part name="TP2" library="testpad" library_urn="urn:adsk.eagle:library:385" deviceset="TP" device="TP10R" package3d_urn="urn:adsk.eagle:package:27959/1"/>
 </parts>
 <sheets>
@@
 </instance>
 <instance part="U2" gate="G$1" x="-254" y="-27.94" smashed="yes"/>
+<instance part="TP2" gate="G$1" x="27.94" y="-12.7" smashed="yes" rot="R270">
+<attribute name="NAME" x="29.21" y="-11.43" size="1.778" layer="95" rot="R270"/>
+<attribute name="TP_SIGNAL_NAME" x="26.67" y="-13.97" size="1.778" layer="97" rot="R270"/>
+</instance>
 </instances>
 <busses>
@@
 <pinref part="U1" gate="G$1" pin="GPIO1"/>
 <wire x1="30.48" y1="30.48" x2="25.4" y2="30.48" width="0.1524" layer="91"/>
-<wire x1="25.4" y1="30.48" x2="25.4" y2="-43.18" width="0.1524" layer="91"/>
+<wire x1="25.4" y1="30.48" x2="25.4" y2="-12.7" width="0.1524" layer="91"/>
 <pinref part="IC1" gate="G$1" pin="PA0"/>
+<wire x1="25.4" y1="-12.7" x2="25.4" y2="-43.18" width="0.1524" layer="91"/>
 <wire x1="25.4" y1="-43.18" x2="5.08" y2="-43.18" width="0.1524" layer="91"/>
+<pinref part="TP2" gate="G$1" pin="TP"/>
+<junction x="25.4" y="-12.7"/>
 </segment>
 </net>
@@
 with this version.
 </note>
+<note version="8.3" severity="warning">
+Since Version 8.3, EAGLE supports URNs for individual library
+assets (packages, symbols, and devices). The URNs of those assets
+will not be understood (or retained) with this version.
+</note>
+<note version="8.3" severity="warning">
+Since Version 8.3, EAGLE supports the association of 3D packages
+with devices in libraries, schematics, and board files. Those 3D
+packages will not be understood (or retained) with this version.
+</note>
 </compatibility>
