File: pcb/v2_experimental/tx_v2.sch (EAGLE design)
At the start: 56 parts, among them IC1 STM32F030F4, IC2 NRF24L01ALT1, SW2 324_SW324_SWITCH_FOOT_HOLE, U2 USBC_16P, U3 MCP73831T-2ACI/OT, U4 XC6206_DEV, Y1 16MHz_12pF

Commit message: new TX header with extra pin
Parts:
- removed IC1: STM32F030F4, exixe_pogo:STM32F030F4
- removed JP1: (no value), adafruit_changed:PINHD-1X3CB
- added IC3: STM32L052K8U66, micro-stm:STM32L052K8U66
- added JP3: (no value), adafruit:PINHD-1X9
- added U$3: PINHD1X4, adafruit_changed:PINHD1X4
Connections:
- removed net N$22: IC1.PF1/OSC_OUT, R7.1, U1.SCL
- removed net N$23: IC1.PF0/OSC_IN, R6.1, U1.SDA
- removed net N$29: IC1.PA3, LED2.A
- new net N$39: R7.1, U1.SCL
- new net N$40: R6.1, U1.SDA
- net +3V3: now also IC3PWR.VDD@1, IC3PWR.VDD@2; no longer IC1.VDD, IC1.VDDA
- net GND: now also IC3PWR.VSS@1; no longer IC1.VSS
- net N$14: no longer IC1.PA7
- net N$15: no longer IC1.PA6
- net N$16: no longer IC1.PA5
- net N$18: no longer IC1.PA10
- net N$20: no longer IC1.PB1
- net N$21: no longer IC1.PA4
- net N$30: no longer IC1.BOOT0
- net N$31: now also U$3.3; no longer IC1.PA13, JP1.3
- net N$32: now also U$3.2; no longer IC1.PA14, JP1.2
- net N$33: now also U$3.1; no longer IC1.PA2, JP1.1
- net N$34: no longer IC1.PA9
- net N$35: no longer IC1.PA1
- net N$36: no longer IC1.PA0

Commit message: hooked up new MCU
Parts:
- removed R14: 1 Ohm, joyAnalog:RESISTOR0805-RES
Connections:
- removed net N$33: U$3.1
- removed net N$34: U2.DN1, U2.DN2
- removed net N$37: C1.1, C14.1, C2.1, IC2.VDD@15, IC2.VDD@18, IC2.VDD@7, R14.2
- new net N$22: IC2.IRQ, IC3MCU.PA15
- new net N$23: IC3MCU.PA3, LED2.A
- new net N$29: IC3MCU.PA13, U$11.1
- new net USB_DM: IC3MCU.PA11, U2.DN1, U2.DN2
- new net USB_DP: IC3MCU.PA12, U2.DP1, U2.DP2
- net +3V3: now also C1.1, C14.1, C2.1, IC2.VDD@15, IC2.VDD@18, IC2.VDD@7, IC3MCU.VDDA, U$3.3; no longer R14.1, U$11.1
- net GND: now also U$3.4; no longer U$11.2
- net N$14: now also IC3MCU.PB5
- net N$15: now also IC3MCU.PB4
- net N$16: now also IC3MCU.PB3
- net N$18: now also IC3MCU.PA14, U$11.2; no longer U2.DP1, U2.DP2
- net N$20: now also IC3MCU.PB6
- net N$21: now also IC3MCU.PC15
- net N$30: now also IC3MCU.BOOT0, IC3MCU.PC14
- net N$31: now also IC3MCU.PA10, U$3.2; no longer U$3.3
- net N$32: now also IC3MCU.PA9, U$3.1; no longer U$3.2
- net N$35: now also IC3MCU.PB1
- net N$36: now also IC3MCU.PA0
- net N$39: now also IC3MCU.PB8
- net N$40: now also IC3MCU.PB7
Other:
- moved on the sheet: IC3, LED2, R12, R13, R9, TP2, U$11, U$3

Commit message: added switch cutout and testpads
Parts:
- removed JP3: (no value), adafruit:PINHD-1X9
- added U$4, U$5, U$6, U$7: TESTPAD, micro-stm:TESTPAD
Connections:
- new net N$33: IC3MCU.PA4, U$5.P$1
- new net N$34: IC3MCU.PA5, U$4.P$1
- new net N$37: IC3MCU.PA6, U$7.P$1
- new net N$41: IC3MCU.PA7, U$6.P$1
Changed lines of the file:
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@@
 <part name="U$2" library="3pos_slide_switch_centered" deviceset="HOT_SWAP_COIN_BAT" device=""/>
 <part name="IC3" library="micro-stm" deviceset="STM32L052K8U6" device="" technology="6"/>
-<part name="JP3" library="adafruit" deviceset="PINHD-1X9" device=""/>
 <part name="U$3" library="adafruit_changed" deviceset="PINHD1X4" device=""/>
 <part name="+3V10" library="supply1" library_urn="urn:adsk.eagle:library:371" deviceset="+3V3" device=""/>
 <part name="GND23" library="supply1" library_urn="urn:adsk.eagle:library:371" deviceset="GND" device=""/>
 <part name="+3V11" library="supply1" library_urn="urn:adsk.eagle:library:371" deviceset="+3V3" device=""/>
+<part name="U$4" library="micro-stm" deviceset="TESTPAD" device=""/>
+<part name="U$6" library="micro-stm" deviceset="TESTPAD" device=""/>
+<part name="U$7" library="micro-stm" deviceset="TESTPAD" device=""/>
+<part name="U$5" library="micro-stm" deviceset="TESTPAD" device=""/>
 </parts>
 <sheets>
@@
 </instance>
 <instance part="IC3" gate="PWR" x="-55.88" y="71.12" smashed="yes"/>
-<instance part="JP3" gate="G$1" x="-347.98" y="-83.82" smashed="yes">
-<attribute name="NAME" x="-354.33" y="-70.485" size="1.778" layer="95"/>
-<attribute name="VALUE" x="-354.33" y="-99.06" size="1.778" layer="96"/>
-</instance>
 <instance part="U$3" gate="1" x="68.58" y="-114.3" smashed="yes" rot="R270">
 <attribute name="NAME" x="76.2" y="-119.38" size="1.27" layer="95" font="vector" rot="R90"/>
@@
 <attribute name="VALUE" x="63.5" y="-99.06" size="1.778" layer="96" rot="R90"/>
 </instance>
+<instance part="U$4" gate="G$1" x="17.78" y="-96.52" smashed="yes"/>
+<instance part="U$6" gate="G$1" x="20.32" y="-91.44" smashed="yes"/>
+<instance part="U$7" gate="G$1" x="20.32" y="-93.98" smashed="yes"/>
+<instance part="U$5" gate="G$1" x="17.78" y="-99.06" smashed="yes"/>
 </instances>
 <busses>
@@
 </segment>
 </net>
+<net name="N$33" class="0">
+<segment>
+<pinref part="IC3" gate="MCU" pin="PA4"/>
+<pinref part="U$5" gate="G$1" pin="P$1"/>
+</segment>
+</net>
+<net name="N$34" class="0">
+<segment>
+<pinref part="IC3" gate="MCU" pin="PA5"/>
+<pinref part="U$4" gate="G$1" pin="P$1"/>
+</segment>
+</net>
+<net name="N$37" class="0">
+<segment>
+<pinref part="U$7" gate="G$1" pin="P$1"/>
+<pinref part="IC3" gate="MCU" pin="PA6"/>
+<wire x1="15.24" y1="-93.98" x2="12.7" y2="-93.98" width="0.1524" layer="91"/>
+</segment>
+</net>
+<net name="N$41" class="0">
+<segment>
+<pinref part="U$6" gate="G$1" pin="P$1"/>
+<pinref part="IC3" gate="MCU" pin="PA7"/>
+<wire x1="15.24" y1="-91.44" x2="12.7" y2="-91.44" width="0.1524" layer="91"/>
+</segment>
+</net>
