File: pcb/v2_experimental/v2_pogo.sch (EAGLE design)
At the start: 2 parts

Commit message: updated pogo board
Parts:
- added JP3: (no value), pinhead:PINHD-1X6
Connections:
- net +3V3: now also JP3.2
- net GND: now also JP3.1
- net N$1: now also JP3.5
- net N$2: now also JP3.4
- net N$5: now also JP3.6
- net N$6: now also JP3.3
Changed lines of the file:
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@@
 <part name="JP2" library="pinhead" library_urn="urn:adsk.eagle:library:325" deviceset="PINHD-1X6" device="" package3d_urn="urn:adsk.eagle:package:22472/2"/>
 <part name="JP1" library="pinhead" library_urn="urn:adsk.eagle:library:325" deviceset="PINHD-1X7" device="" package3d_urn="urn:adsk.eagle:package:22477/2"/>
+<part name="JP3" library="pinhead" library_urn="urn:adsk.eagle:library:325" deviceset="PINHD-1X6" device="" package3d_urn="urn:adsk.eagle:package:22472/2"/>
+<part name="GND1" library="clock" deviceset="GND" device=""/>
+<part name="+3V1" library="supply1" library_urn="urn:adsk.eagle:library:371" deviceset="+3V3" device=""/>
 </parts>
 <sheets>
@@
 <attribute name="VALUE" x="16.51" y="-35.56" size="1.778" layer="96"/>
 </instance>
+<instance part="JP3" gate="A" x="22.86" y="-50.8" smashed="yes">
+<attribute name="NAME" x="16.51" y="-40.005" size="1.778" layer="95"/>
+<attribute name="VALUE" x="16.51" y="-60.96" size="1.778" layer="96"/>
+</instance>
+<instance part="GND1" gate="1" x="30.48" y="-45.72" smashed="yes">
+<attribute name="VALUE" x="27.94" y="-48.26" size="1.778" layer="96"/>
+</instance>
+<instance part="+3V1" gate="G$1" x="10.16" y="-40.64" smashed="yes">
+<attribute name="VALUE" x="7.62" y="-45.72" size="1.778" layer="96" rot="R90"/>
+</instance>
 </instances>
 <busses>
@@
 <pinref part="JP1" gate="A" pin="7"/>
 <wire x1="-2.54" y1="-33.02" x2="20.32" y2="-33.02" width="0.1524" layer="91"/>
+<pinref part="JP3" gate="A" pin="5"/>
+<wire x1="-2.54" y1="-33.02" x2="-2.54" y2="-53.34" width="0.1524" layer="91"/>
+<wire x1="-2.54" y1="-53.34" x2="20.32" y2="-53.34" width="0.1524" layer="91"/>
+<junction x="-2.54" y="-33.02"/>
 </segment>
 </net>
@@
 <pinref part="JP1" gate="A" pin="6"/>
 <wire x1="-2.54" y1="-30.48" x2="20.32" y2="-30.48" width="0.1524" layer="91"/>
+<wire x1="-2.54" y1="-30.48" x2="-5.08" y2="-30.48" width="0.1524" layer="91"/>
+<junction x="-2.54" y="-30.48"/>
+<pinref part="JP3" gate="A" pin="4"/>
+<wire x1="-5.08" y1="-30.48" x2="-5.08" y2="-50.8" width="0.1524" layer="91"/>
+<wire x1="-5.08" y1="-50.8" x2="20.32" y2="-50.8" width="0.1524" layer="91"/>
 </segment>
 </net>
@@
 <pinref part="JP1" gate="A" pin="2"/>
 <wire x1="7.62" y1="-20.32" x2="20.32" y2="-20.32" width="0.1524" layer="91"/>
+<wire x1="20.32" y1="-20.32" x2="40.64" y2="-20.32" width="0.1524" layer="91"/>
+<junction x="20.32" y="-20.32"/>
+<pinref part="JP3" gate="A" pin="6"/>
+<wire x1="40.64" y1="-20.32" x2="40.64" y2="-55.88" width="0.1524" layer="91"/>
+<wire x1="40.64" y1="-55.88" x2="20.32" y2="-55.88" width="0.1524" layer="91"/>
 </segment>
 </net>
@@
 <pinref part="JP1" gate="A" pin="1"/>
 <wire x1="5.08" y1="-17.78" x2="20.32" y2="-17.78" width="0.1524" layer="91"/>
+<wire x1="20.32" y1="-17.78" x2="38.1" y2="-17.78" width="0.1524" layer="91"/>
+<wire x1="38.1" y1="-17.78" x2="38.1" y2="-48.26" width="0.1524" layer="91"/>
+<junction x="20.32" y="-17.78"/>
+<pinref part="JP3" gate="A" pin="3"/>
+<wire x1="38.1" y1="-48.26" x2="20.32" y2="-48.26" width="0.1524" layer="91"/>
 </segment>
 </net>
@@
 <junction x="-2.54" y="-27.94"/>
 </segment>
+<segment>
+<pinref part="JP3" gate="A" pin="1"/>
+<pinref part="GND1" gate="1" pin="GND"/>
+<wire x1="20.32" y1="-43.18" x2="30.48" y2="-43.18" width="0.1524" layer="91"/>
+</segment>
 </net>
 <net name="+3V3" class="0">
@@
 <junction x="-2.54" y="-25.4"/>
 </segment>
+<segment>
+<pinref part="+3V1" gate="G$1" pin="+3V3"/>
+<wire x1="10.16" y1="-43.18" x2="10.16" y2="-45.72" width="0.1524" layer="91"/>
+<pinref part="JP3" gate="A" pin="2"/>
+<wire x1="10.16" y1="-45.72" x2="20.32" y2="-45.72" width="0.1524" layer="91"/>
+</segment>
 </net>
